Commit message: Stance

File: robots/b1.urdf (robot description, URDF)
Before this commit: robot b1_description, 19 links, 18 joints
Links:
- added link FL_calf_rotor, mass 0.266; collision cylinder length=0.02 radius=0.05; visual cylinder length=0.02 radius=0.05
- added link FL_hip_rotor, mass 0.199; collision cylinder length=0.02 radius=0.05; visual cylinder length=0.02 radius=0.05
- added link FL_thigh_rotor, mass 0.266; collision cylinder length=0.02 radius=0.05; visual cylinder length=0.02 radius=0.05
- added link FR_calf_rotor, mass 0.266; collision cylinder length=0.02 radius=0.05; visual cylinder length=0.02 radius=0.05
- added link FR_hip_rotor, mass 0.199; collision cylinder length=0.02 radius=0.05; visual cylinder length=0.02 radius=0.05
- added link FR_thigh_rotor, mass 0.266; collision cylinder length=0.02 radius=0.05; visual cylinder length=0.02 radius=0.05
- added link RL_calf_rotor, mass 0.266; collision cylinder length=0.02 radius=0.05; visual cylinder length=0.02 radius=0.05
- added link RL_hip_rotor, mass 0.199; collision cylinder length=0.02 radius=0.05; visual cylinder length=0.02 radius=0.05
- added link RL_thigh_rotor, mass 0.266; collision cylinder length=0.02 radius=0.05; visual cylinder length=0.02 radius=0.05
- added link RR_calf_rotor, mass 0.266; collision cylinder length=0.02 radius=0.05; visual cylinder length=0.02 radius=0.05
- added link RR_hip_rotor, mass 0.199; collision cylinder length=0.02 radius=0.05; visual cylinder length=0.02 radius=0.05
- added link RR_thigh_rotor, mass 0.266; collision cylinder length=0.02 radius=0.05; visual cylinder length=0.02 radius=0.05
- link FL_calf: mass 0.207 -> 0.857; geometry collision box size=0.35 0.04 0.05; visual mesh filename=package://b1_description/meshes/calf.dae scale=1 1 1
- link FL_foot: mass 0.06 -> 0.05
- link FL_hip: mass 1.993 -> 2.1
- link FL_thigh: mass 0.639 -> 3.934
- link FR_calf: mass 0.207 -> 0.857; geometry collision box size=0.35 0.04 0.05; visual mesh filename=package://b1_description/meshes/calf.dae scale=1 1 1
- link FR_foot: mass 0.06 -> 0.05
- link FR_hip: mass 1.993 -> 2.1
- link FR_thigh: mass 0.639 -> 3.934
- link RL_calf: mass 0.207 -> 0.857; geometry collision box size=0.35 0.04 0.05; visual mesh filename=package://b1_description/meshes/calf.dae scale=1 1 1
- link RL_foot: mass 0.06 -> 0.05
- link RL_hip: mass 1.993 -> 2.1
- link RL_thigh: mass 0.639 -> 3.934
- link RR_calf: mass 0.207 -> 0.857; geometry collision box size=0.35 0.04 0.05; visual mesh filename=package://b1_description/meshes/calf.dae scale=1 1 1
- link RR_foot: mass 0.06 -> 0.05
- link RR_hip: mass 1.993 -> 2.1
- link RR_thigh: mass 0.639 -> 3.934
- link base: mass 50 -> None
- link trunk: mass 9.041 -> 25
Joints:
- added joint FL_calf_rotor_joint: type fixed, parent FL_thigh, child FL_calf_rotor, origin xyz=0.0 -0.0519 0 rpy=0 0 0
- added joint FL_hip_rotor_joint: type fixed, parent trunk, child FL_hip_rotor, origin xyz=0.1955 0.072 0 rpy=0 0 0
- added joint FL_thigh_rotor_joint: type fixed, parent FL_hip, child FL_thigh_rotor, origin xyz=0.0 0.00935 0 rpy=0 0 0
- added joint FR_calf_rotor_joint: type fixed, parent FR_thigh, child FR_calf_rotor, origin xyz=0.0 0.0519 0 rpy=0 0 0
- added joint FR_hip_rotor_joint: type fixed, parent trunk, child FR_hip_rotor, origin xyz=0.1955 -0.072 0 rpy=0 0 0
- added joint FR_thigh_rotor_joint: type fixed, parent FR_hip, child FR_thigh_rotor, origin xyz=0.0 -0.00935 0 rpy=0 0 0
- added joint RL_calf_rotor_joint: type fixed, parent RL_thigh, child RL_calf_rotor, origin xyz=0.0 -0.0519 0 rpy=0 0 0
- added joint RL_hip_rotor_joint: type fixed, parent trunk, child RL_hip_rotor, origin xyz=-0.1955 0.072 0 rpy=0 0 0
- added joint RL_thigh_rotor_joint: type fixed, parent RL_hip, child RL_thigh_rotor, origin xyz=0.0 0.00935 0 rpy=0 0 0
- added joint RR_calf_rotor_joint: type fixed, parent RR_thigh, child RR_calf_rotor, origin xyz=0.0 0.0519 0 rpy=0 0 0
- added joint RR_hip_rotor_joint: type fixed, parent trunk, child RR_hip_rotor, origin xyz=-0.1955 -0.072 0 rpy=0 0 0
- added joint RR_thigh_rotor_joint: type fixed, parent RR_hip, child RR_thigh_rotor, origin xyz=0.0 -0.00935 0 rpy=0 0 0
- joint FL_calf_joint: limit lower=-2.6 upper=-0.6 effort=100 velocity=20 -> lower=-2.6 upper=-0.6 effort=140 velocity=15.55
- joint FL_hip_joint: limit lower=-0.75 upper=0.75 effort=100 velocity=20 -> lower=-0.75 upper=0.75 effort=91.0035 velocity=19.69
- joint FL_thigh_joint: limit lower=-1.0 upper=3.5 effort=100 velocity=20 -> lower=-1.0 upper=3.5 effort=93.33 velocity=23.32; type continuous -> revolute
- joint FR_calf_joint: limit lower=-2.6 upper=-0.6 effort=100 velocity=20 -> lower=-2.6 upper=-0.6 effort=140 velocity=15.55
- joint FR_hip_joint: limit lower=-0.75 upper=0.75 effort=100 velocity=20 -> lower=-0.75 upper=0.75 effort=91.0035 velocity=19.69
- joint FR_thigh_joint: limit lower=-1.0 upper=3.5 effort=100 velocity=20 -> lower=-1.0 upper=3.5 effort=93.33 velocity=23.32; type continuous -> revolute
- joint RL_calf_joint: limit lower=-2.6 upper=-0.6 effort=100 velocity=20 -> lower=-2.6 upper=-0.6 effort=140 velocity=15.55
- joint RL_hip_joint: limit lower=-0.75 upper=0.75 effort=100 velocity=20 -> lower=-0.75 upper=0.75 effort=91.0035 velocity=19.69
- joint RL_thigh_joint: limit lower=-1.0 upper=3.5 effort=100 velocity=20 -> lower=-1.0 upper=3.5 effort=93.33 velocity=23.32; type continuous -> revolute
- joint RR_calf_joint: limit lower=-2.6 upper=-0.6 effort=100 velocity=20 -> lower=-2.6 upper=-0.6 effort=140 velocity=15.55
- joint RR_hip_joint: limit lower=-0.75 upper=0.75 effort=100 velocity=20 -> lower=-0.75 upper=0.75 effort=91.0035 velocity=19.69
- joint RR_thigh_joint: limit lower=-1.0 upper=3.5 effort=100 velocity=20 -> lower=-1.0 upper=3.5 effort=93.33 velocity=23.32; type continuous -> revolute

File: robots/b1_description/xacro/const.xacro (robot description, xacro)
@@ -28,4 +28,23 @@
     <xacro:property name="trunk_offset_z" value="0.01675"/>
     <xacro:property name="hip_offset" value="0.12675"/>
+    <!-- offset of link and rotor locations (left front) -->
+    <xacro:property name="hip_offset_x" value="0.3455"/>
+    <xacro:property name="hip_offset_y" value="0.072"/>
+    <xacro:property name="hip_offset_z" value="0.0"/>
+    <xacro:property name="hip_rotor_offset_x" value="0.1955"/>
+    <xacro:property name="hip_rotor_offset_y" value="0.072"/>
+    <xacro:property name="hip_rotor_offset_z" value="0.0"/>
+    <xacro:property name="thigh_offset_x" value="0"/>
+    <xacro:property name="thigh_offset_y" value="0.12675"/>
+    <xacro:property name="thigh_offset_z" value="0.0"/>
+    <xacro:property name="thigh_rotor_offset_x" value="0.0"/>
+    <xacro:property name="thigh_rotor_offset_y" value="0.00935"/>
+    <xacro:property name="thigh_rotor_offset_z" value="0.0"/>
+    <xacro:property name="calf_offset_x" value="0.0"/>
+    <xacro:property name="calf_offset_y" value="0.0"/>
+    <xacro:property name="calf_offset_z" value="-0.35"/>
+    <xacro:property name="calf_rotor_offset_x" value="0.0"/>
+    <xacro:property name="calf_rotor_offset_y" value="-0.0519"/>
+    <xacro:property name="calf_rotor_offset_z" value="0.0"/>
     <!-- joint limits -->
     <xacro:property name="damping" value="0"/>
@@ -33,59 +52,89 @@
     <xacro:property name="hip_position_max" value="0.75"/>
     <xacro:property name="hip_position_min" value="-0.75"/>
-    <xacro:property name="hip_velocity_max" value="20"/>
-    <xacro:property name="hip_torque_max" value="100"/>
+    <xacro:property name="hip_velocity_max" value="19.69"/>
+    <xacro:property name="hip_torque_max" value="91.0035"/>
     <xacro:property name="thigh_position_max" value="3.5"/>
     <xacro:property name="thigh_position_min" value="-1.0"/>
-    <xacro:property name="thigh_velocity_max" value="20"/>
-    <xacro:property name="thigh_torque_max" value="100"/>
+    <xacro:property name="thigh_velocity_max" value="23.32"/>
+    <xacro:property name="thigh_torque_max" value="93.33"/>
     <xacro:property name="calf_position_max" value="-0.6"/>
     <xacro:property name="calf_position_min" value="-2.6"/>
-    <xacro:property name="calf_velocity_max" value="20"/>
-    <xacro:property name="calf_torque_max" value="100"/>
+    <xacro:property name="calf_velocity_max" value="15.55"/>
+    <xacro:property name="calf_torque_max" value="140"/>
     <!-- dynamics inertial value -->
     <!-- trunk -->
-    <xacro:property name="trunk_mass" value="18.276"/>
-    <xacro:property name="trunk_com_x" value="-0.01"/>
-    <xacro:property name="trunk_com_y" value="0.0"/>
-    <xacro:property name="trunk_com_z" value="0.00"/>
-    <xacro:property name="trunk_ixx" value="0.174426"/>
-    <xacro:property name="trunk_ixy" value="0.005544"/>
-    <xacro:property name="trunk_ixz" value="0.003278"/>
-    <xacro:property name="trunk_iyy" value="0.700100"/>
-    <xacro:property name="trunk_iyz" value="0.000007"/>
-    <xacro:property name="trunk_izz" value="0.785955"/>
+    <xacro:property name="trunk_mass" value="25"/>
+    <xacro:property name="trunk_com_x" value="0.008987"/>
+    <xacro:property name="trunk_com_y" value="0.002243"/>
+    <xacro:property name="trunk_com_z" value="0.003013"/>
+    <xacro:property name="trunk_ixx" value="0.183142146"/>
+    <xacro:property name="trunk_ixy" value="-0.001379002"/>
+    <xacro:property name="trunk_ixz" value="-0.027956055"/>
+    <xacro:property name="trunk_iyy" value="0.756327752"/>
+    <xacro:property name="trunk_iyz" value="0.000193774"/>
+    <xacro:property name="trunk_izz" value="0.783777558"/>
     <!-- hip (left front) -->
-    <xacro:property name="hip_mass" value="1.998"/>
+    <xacro:property name="hip_mass" value="2.1"/>
     <xacro:property name="hip_com_x" value="-0.020298"/>
-    <xacro:property name="hip_com_y" value="-0.009758"/>
-    <xacro:property name="hip_com_z" value="-0.000109"/>
-    <xacro:property name="hip_ixx" value="0.004066"/>
-    <xacro:property name="hip_ixy" value="-0.000288"/>
-    <xacro:property name="hip_ixz" value="0.000000"/>
-    <xacro:property name="hip_iyy" value="0.008775"/>
-    <xacro:property name="hip_iyz" value="-0.000000"/>
-    <xacro:property name="hip_izz" value="0.006060"/>
+    <xacro:property name="hip_com_y" value="0.009758"/>
+    <xacro:property name="hip_com_z" value="0.000109"/>
+    <xacro:property name="hip_ixx" value="0.00406608"/>
+    <xacro:property name="hip_ixy" value="-0.000288071"/>
+    <xacro:property name="hip_ixz" value="-0.000004371"/>
+    <xacro:property name="hip_iyy" value="0.008775259"/>
+    <xacro:property name="hip_iyz" value="0.000001811"/>
+    <xacro:property name="hip_izz" value="0.006060348"/>
+    <xacro:property name="hip_rotor_mass" value="0.199"/>
+    <xacro:property name="hip_rotor_com_x" value="0.0"/>
+    <xacro:property name="hip_rotor_com_y" value="0.0"/>
+    <xacro:property name="hip_rotor_com_z" value="0.0"/>
+    <xacro:property name="hip_rotor_ixx" value="0.00039249"/>
+    <xacro:property name="hip_rotor_ixy" value="0.0"/>
+    <xacro:property name="hip_rotor_ixz" value="0.0"/>
+    <xacro:property name="hip_rotor_iyy" value="0.000219397"/>
+    <xacro:property name="hip_rotor_iyz" value="0.0"/>
+    <xacro:property name="hip_rotor_izz" value="0.000219397"/>
     <!-- thigh -->
-    <xacro:property name="thigh_mass" value="3.444"/>
-    <xacro:property name="thigh_com_x" value="0.0050"/>
-    <xacro:property name="thigh_com_y" value="-0.0250"/>
-    <xacro:property name="thigh_com_z" value="-0.0512"/>
-    <xacro:property name="thigh_ixx" value="0.035982"/>
-    <xacro:property name="thigh_ixy" value="0.000032"/>
-    <xacro:property name="thigh_ixz" value="0.001385"/>
-    <xacro:property name="thigh_iyy" value="0.037758"/>
-    <xacro:property name="thigh_iyz" value="-0.004234"/>
-    <xacro:property name="thigh_izz" value="0.006637"/>
+    <xacro:property name="thigh_mass" value="3.934"/>
+    <xacro:property name="thigh_com_x" value="-0.000235"/>
+    <xacro:property name="thigh_com_y" value="-0.028704"/>
+    <xacro:property name="thigh_com_z" value="-0.054169"/>
+    <xacro:property name="thigh_ixx" value="0.044459086"/>
+    <xacro:property name="thigh_ixy" value="0.000128738"/>
+    <xacro:property name="thigh_ixz" value="-0.002343913"/>
+    <xacro:property name="thigh_iyy" value="0.046023457"/>
+    <xacro:property name="thigh_iyz" value="0.006032996"/>
+    <xacro:property name="thigh_izz" value="0.008696078"/>
+    <xacro:property name="thigh_rotor_mass" value="0.266"/>
+    <xacro:property name="thigh_rotor_com_x" value="0.0"/>
+    <xacro:property name="thigh_rotor_com_y" value="0.0"/>
+    <xacro:property name="thigh_rotor_com_z" value="0.0"/>
+    <xacro:property name="thigh_rotor_ixx" value="0.000485657"/>
+    <xacro:property name="thigh_rotor_ixy" value="0.0"/>
+    <xacro:property name="thigh_rotor_ixz" value="0.0"/>
+    <xacro:property name="thigh_rotor_iyy" value="0.00091885"/>
+    <xacro:property name="thigh_rotor_iyz" value="0.0"/>
+    <xacro:property name="thigh_rotor_izz" value="0.000485657"/>
     <!-- calf -->
-    <xacro:property name="calf_mass" value="0.803"/>
-    <xacro:property name="calf_com_x" value="0.00565"/>
-    <xacro:property name="calf_com_y" value="-0.000236"/>
-    <xacro:property name="calf_com_z" value="-0.150538"/>
-    <xacro:property name="calf_ixx" value="0.017617"/>
-    <xacro:property name="calf_ixy" value="0.000000"/>
-    <xacro:property name="calf_ixz" value="-0.000532"/>
-    <xacro:property name="calf_iyy" value="0.017722"/>
-    <xacro:property name="calf_iyz" value="-0.000030"/>
-    <xacro:property name="calf_izz" value="0.000409"/>
+    <xacro:property name="calf_mass" value="0.857"/>
+    <xacro:property name="calf_com_x" value="0.005237"/>
+    <xacro:property name="calf_com_y" value="0.0"/>
+    <xacro:property name="calf_com_z" value="-0.202805"/>
+    <xacro:property name="calf_ixx" value="0.015011003"/>
+    <xacro:property name="calf_ixy" value="0.000000052"/>
+    <xacro:property name="calf_ixz" value="0.000250042"/>
+    <xacro:property name="calf_iyy" value="0.015159462"/>
+    <xacro:property name="calf_iyz" value="0.000000461"/>
+    <xacro:property name="calf_izz" value="0.000375749"/>
+    <xacro:property name="calf_rotor_mass" value="0.266"/>
+    <xacro:property name="calf_rotor_com_x" value="0.0"/>
+    <xacro:property name="calf_rotor_com_y" value="0.0"/>
+    <xacro:property name="calf_rotor_com_z" value="0.0"/>
+    <xacro:property name="calf_rotor_ixx" value="0.000485657"/>
+    <xacro:property name="calf_rotor_ixy" value="0.0"/>
+    <xacro:property name="calf_rotor_ixz" value="0.0"/>
+    <xacro:property name="calf_rotor_iyy" value="0.00091885"/>
+    <xacro:property name="calf_rotor_iyz" value="0.0"/>
+    <xacro:property name="calf_rotor_izz" value="0.000485657"/>
     <!-- foot -->
     <xacro:property name="foot_mass" value="0.05"/>

File: robots/b1_description/xacro/robot.xacro (robot description, xacro)
@@ -5,6 +5,6 @@
     <xacro:include filename="$(find b1_description)/xacro/leg.xacro"/>
     <xacro:include filename="$(find b1_description)/xacro/gazebo.xacro"/>
-    <!-- Rollover Protection mode will add an additional stick on the top, use "true" or "false" to switch it. -->
-    <xacro:property name="rolloverProtection" value="false"/>
+    <!-- Rotor related joint and link is only for demonstrate location. -->
+    <!-- Actually, the rotor will rotate and the joint is not fixed. Reduction ratio should be considered. -->
     <!-- Debug mode will hung up the robot, use "true" or "false" to switch it. -->
     <!-- <xacro:if value="$(arg DEBUG)">
@@ -58,33 +58,4 @@
         </inertial>
     </link>
-    <xacro:if value="${(rolloverProtection == 'true')}">
-        <joint name="stick_joint" type="fixed">
-            <parent link="trunk"/>
-            <child link="stick_link"/>
-            <origin rpy="0 0 0" xyz="${0.18} 0 ${stick_length/2.0+0.08}"/>
-        </joint>
-        <link name="stick_link">
-            <visual>
-                <geometry>
-                    <cylinder length="${stick_length}" radius="${stick_radius}"/>
-                </geometry>
-                <origin rpy="0 0 0" xyz="0 0 0"/>
-                <material name="white"/>
-            </visual>
-            <collision>
-                <geometry>
-                    <cylinder length="${stick_length}" radius="${stick_radius}"/>
-                </geometry>
-                <origin rpy="0 0 0" xyz="0 0 0"/>
-            </collision>
-            <inertial>
-                <mass value="${stick_mass}"/>
-                <inertia
-                    ixx="${stick_mass / 2.0 * (stick_radius*stick_radius)}" ixy="0.0" ixz="0.0"
-                    iyy="${stick_mass / 12.0 * (3*stick_radius*stick_radius + stick_length*stick_length)}" iyz="0.0"
-                    izz="${stick_mass / 12.0 * (3*stick_radius*stick_radius + stick_length*stick_length)}"/>
-            </inertial>
-        </link>
-    </xacro:if>
     <joint name="imu_joint" type="fixed">
         <parent link="trunk"/>
@@ -96,5 +67,5 @@
             <mass value="0.001"/>
             <origin rpy="0 0 0" xyz="0 0 0"/>
-            <inertia ixx="0.0001" ixy="0" ixz="0" iyy="0.000001" iyz="0" izz="0.0001"/>
+            <inertia ixx="0.0001" ixy="0" ixz="0" iyy="0.0001" iyz="0" izz="0.0001"/>
         </inertial>
         <visual>
@@ -112,16 +83,8 @@
         </collision>
     </link>
-    <xacro:leg name="FR" mirror="-1" mirror_dae= "False" front_hind="1" front_hind_dae="True">
-        <origin rpy="0 0 0" xyz="${leg_offset_x} ${-leg_offset_y} 0"/>
-    </xacro:leg>
-    <xacro:leg name="FL" mirror="1" mirror_dae="True" front_hind="1" front_hind_dae="True">
-        <origin rpy="0 0 0" xyz="${leg_offset_x} ${leg_offset_y} 0"/>
-    </xacro:leg>
-    <xacro:leg name="RR" mirror="-1" mirror_dae="False" front_hind="-1" front_hind_dae="False">
-        <origin rpy="0 0 0" xyz="${-leg_offset_x} ${-leg_offset_y} 0"/>
-    </xacro:leg>
-    <xacro:leg name="RL" mirror="1" mirror_dae="True" front_hind="-1" front_hind_dae="False">
-        <origin rpy="0 0 0" xyz="${-leg_offset_x} ${leg_offset_y} 0"/>
-    </xacro:leg>
+    <xacro:leg name="FR" mirror="-1" mirror_dae= "False" front_hind="1"  front_hind_dae="True"  />
+    <xacro:leg name="FL" mirror="1"  mirror_dae="True"   front_hind="1"  front_hind_dae="True"  />
+    <xacro:leg name="RR" mirror="-1" mirror_dae="False"  front_hind="-1" front_hind_dae="False" />
+    <xacro:leg name="RL" mirror="1"  mirror_dae="True"   front_hind="-1" front_hind_dae="False" />
     <!-- <xacro:stairs stairs="15" xpos="0" ypos="2.0" zpos="0" /> -->
 </robot>
